File: ceiling-light-controller/hardware/hardware.sch (KiCad schematic (older format))
At the start: 18 parts, among them Q1 BT136-500, T1 Transformer_1P_1S, U1 LTV-817, U2 L7805, U3 MOC3021M, U4 WeMos_mini

Commit message: small changes
Parts:
- added J1: Screw_Terminal_01x03, symbol Connector:Screw_Terminal_01x03
- added J2: Screw_Terminal_01x02, symbol Connector:Screw_Terminal_01x02
Connections:
- wire segments 70 -> 81
Other:
- moved on the sheet: Q1, U3
