File: ceiling-light-controller/hardware/ceiling-light-controller.sch (KiCad schematic (older format))
At the start: 20 parts, among them J1 Screw_Terminal_01x03, J2 Screw_Terminal_01x02, Q1 BT136-500, T1 Transformer_1P_1S, U1 LTV-817, U2 L7805, U3 MOC3021M, U4 WeMos_mini

Commit message: renaming
Parts:
- removed C3, C4: 0.1µf, symbol Device:C
- removed U2: L7805, symbol Regulator_Linear:L7805
- added U5: DSN-MINI-360, symbol made-in-china:DSN-MINI-360
Connections:
- wire segments 81 -> 76
Changed lines of the file:
@@
-$EndComp
-$Comp
-L Device:CP C2
-U 1 1 5CD36E4A
-P 3400 2100
-F 0 "C2" H 3250 2400 50  0000 L CNN
-F 1 "470µf" H 3250 2300 50  0000 L CNN
-F 2 "" H 3438 1950 50  0001 C CNN
-F 3 "~" H 3400 2100 50  0001 C CNN
-	1    3400 2100
-	1    0    0    -1
-$EndComp
-$Comp
-L Regulator_Linear:L7805 U2
-U 1 1 5CD36F79
-P 4200 1950
-F 0 "U2" H 4200 2192 50  0000 C CNN
-F 1 "L7805" H 4200 2101 50  0000 C CNN
-F 2 "" H 4225 1800 50  0001 L CIN
-F 3 "http://www.st.com/content/ccc/resource/technical/document/datasheet/41/4f/b3/b0/12/d4/47/88/CD00000444.pdf/files/CD00000444.pdf/jcr:content/translations/en.CD00000444.pdf" H 4200 1900 50  0001 C CNN
-	1    4200 1950
-	1    0    0    -1
 $EndComp
 $Comp
@@
 $EndComp
 $Comp
-L Device:C C3
-U 1 1 5CD37F4F
-P 3700 2100
-F 0 "C3" H 3600 2400 50  0000 L CNN
-F 1 "0.1µf" H 3600 2300 50  0000 L CNN
-F 2 "" H 3738 1950 50  0001 C CNN
-F 3 "~" H 3700 2100 50  0001 C CNN
-	1    3700 2100
-	1    0    0    -1
-$EndComp
-$Comp
-L Device:C C4
-U 1 1 5CD37FCF
-P 4600 2100
-F 0 "C4" H 4715 2146 50  0000 L CNN
-F 1 "0.1µf" H 4715 2055 50  0000 L CNN
-F 2 "" H 4638 1950 50  0001 C CNN
-F 3 "~" H 4600 2100 50  0001 C CNN
-	1    4600 2100
-	1    0    0    -1
-$EndComp
-$Comp
 L power:VAC #PWR0104
 U 1 1 5CD3818E
@@
 F 0 "U4" H 5600 2687 60  0000 C CNN
 F 1 "WeMos_mini" H 5600 2581 60  0000 C CNN
-F 2 "" H 6150 1350 60  0000 C CNN
+F 2 "" H 6150 1350 60  0001 C CNN
 F 3 "http://www.wemos.cc/Products/d1_mini.html" H 5600 2581 60  0001 C CNN
 	1    5600 2050
@@
 Wire Wire Line
 	2550 2600 2950 2600
-Wire Wire Line
-	4200 2300 4200 2250
-Wire Wire Line
-	4500 1950 4600 1950
 $Comp
 L power:GND #PWR0107
@@
 L power:GND #PWR0108
 U 1 1 5CD4B718
-P 4600 2350
-F 0 "#PWR0108" H 4600 2100 50  0001 C CNN
-F 1 "GND" H 4605 2177 50  0000 C CNN
-F 2 "" H 4600 2350 50  0001 C CNN
-F 3 "" H 4600 2350 50  0001 C CNN
-	1    4600 2350
-	1    0    0    -1
-$EndComp
-Connection ~ 4200 2300
-Wire Wire Line
-	4200 2300 4600 2300
-Wire Wire Line
-	4600 2300 4600 2250
-Wire Wire Line
-	3400 1950 3700 1950
+P 4000 2350
+F 0 "#PWR0108" H 4000 2100 50  0001 C CNN
+F 1 "GND" H 4005 2177 50  0000 C CNN
+F 2 "" H 4000 2350 50  0001 C CNN
+F 3 "" H 4000 2350 50  0001 C CNN
+	1    4000 2350
+	1    0    0    -1
+$EndComp
 Wire Wire Line
 	3250 2300 3400 2300
 Wire Wire Line
-	3700 2300 3700 2250
-Connection ~ 3700 2300
-Wire Wire Line
-	3700 2300 4200 2300
-Wire Wire Line
 	3400 2300 3400 2250
-Connection ~ 3400 2300
-Wire Wire Line
-	3400 2300 3700 2300
-Wire Wire Line
-	3700 1950 3900 1950
-Connection ~ 3700 1950
-Wire Wire Line
-	4600 2300 4600 2350
-Connection ~ 4600 2300
-Wire Wire Line
-	3400 1950 2650 1950
 Wire Wire Line
 	2650 1950 2650 2300
-Connection ~ 3400 1950
 Wire Wire Line
 	1800 2750 1800 2850
@@
 	1550 2500 1550 2750
 Wire Wire Line
-	4600 1950 4600 1700
-Connection ~ 4600 1950
-Connection ~ 4600 1700
-Wire Wire Line
 	1650 2100 1650 3450
 Wire Wire Line
@@
 Wire Wire Line
 	1650 3550 1800 3550
+Wire Wire Line
+	3400 1950 2650 1950
+$Comp
+L Device:CP C2
+U 1 1 5CD36E4A
+P 3400 2100
+F 0 "C2" H 3250 2400 50  0000 L CNN
+F 1 "470µf" H 3250 2300 50  0000 L CNN
+F 2 "" H 3438 1950 50  0001 C CNN
+F 3 "~" H 3400 2100 50  0001 C CNN
+	1    3400 2100
+	1    0    0    -1
+$EndComp
+Wire Wire Line
+	4000 2300 4000 2350
+$Comp
+L made-in-china:DSN-MINI-360 U5
+U 1 1 5CD70C62
+P 3850 1850
+F 0 "U5" H 4000 1900 50  0000 C CNN
+F 1 "DSN-MINI-360" H 4250 2000 50  0000 C CNN
+F 2 "" H 3850 1550 50  0001 C CNN
+F 3 "" H 3850 1550 50  0001 C CNN
+	1    3850 1850
+	1    0    0    -1
+$EndComp
+Wire Wire Line
+	3400 1950 3750 1950
+Connection ~ 3400 1950
+Wire Wire Line
+	3400 2300 4000 2300
+Wire Wire Line
+	4000 2300 4000 2150
+Connection ~ 3400 2300
+Wire Wire Line
+	4250 1950 4600 1950
+Wire Wire Line
+	4600 1950 4600 1700
+Connection ~ 4600 1700
+Connection ~ 4000 2300
 $EndSCHEMATC

Commit message: new AD-DC conv; footprint refs; simple PCB
Parts:
- removed C2: 470µf, symbol Device:CP
- removed D1, D2: D_Bridge_+-AA, symbol Device:D_Bridge_+-AA
- removed T1: Transformer_1P_1S, symbol Device:Transformer_1P_1S
- removed U5: DSN-MINI-360, symbol made-in-china:DSN-MINI-360
- added BR1: DB107-BP, DB107-BP:DIP825W56P510L828H330Q4N, symbol DB107-BP:DB107-BP
- added U2: HLK-PM03, Power_Supply:HLK-PM01, symbol Power_Supplies:HLK-PM03
- C1, C5: footprint (none) -> Capacitor_THT:CP_Axial_L10.0mm_D4.5mm_P15.00mm_Horizontal
- J1: footprint (none) -> TerminalBlock:TerminalBlock_bornier-3_P5.08mm
- J2: footprint (none) -> TerminalBlock:TerminalBlock_bornier-2_P5.08mm
- R1, R2, R3, R4, R5: footprint (none) -> Resistor_THT:R_Axial_DIN0309_L9.0mm_D3.2mm_P12.70mm_Horizontal
- U3: footprint (none) -> Package_DIP:DIP-6_W7.62mm
- U4: footprint (none) -> wemos-d1-mini:wemos-d1-mini-embedded
Connections:
- wire segments 76 -> 59
Other:
- moved on the sheet: Q1, U3

Commit message: LED, LDR; PCB layout; copper traces
Parts:
- added D1: WS2812B, LED_SMD:LED_WS2812B_PLCC4_5.0x5.0mm_P3.2mm, symbol LED:WS2812B
- added R6: 10000, Resistor_THT:R_Axial_DIN0309_L9.0mm_D3.2mm_P12.70mm_Horizontal, symbol Device:R
- added R7: LDR03, OptoDevice:R_LDR_10x8.5mm_P7.6mm_Vertical, symbol Sensor_Optical:LDR03
- C1: footprint Capacitor_THT:CP_Axial_L10.0mm_D4.5mm_P15.00mm_Horizontal -> Capacitor_THT:CP_Radial_D4.0mm_P1.50mm
- C5: footprint Capacitor_THT:CP_Axial_L10.0mm_D4.5mm_P15.00mm_Horizontal -> Capacitor_THT:C_Disc_D5.1mm_W3.2mm_P5.00mm
- Q1: footprint Package_TO_SOT_THT:TO-220-3_Vertical -> slimc:TO-220-3_Vertical_Triode_Heatsink
Connections:
- net labels removed: NEUT, VAC
- wire segments 59 -> 62
