File: ceiling-light-controller/hardware/ceiling-light-controller.kicad_pcb (KiCad board)
At the start: 2 copper layers, 90.5 x 83 mm, 18 parts, among them J1 Screw_Terminal_01x03, J2 Screw_Terminal_01x02, Q1 BT136-500, U1 LTV-817, U2 HLK-PM03, U3 MOC3021M, U4 WeMos_mini

Commit message: moved submodules
Routing:
- net Net-(J1-Pad1): track 110.8 -> 160.0 mm
- net Net-(C5-Pad2): track 29.4 -> 58.8 mm
- net Net-(BR1-Pad4): track 114.8 -> 142.0 mm
- net Net-(C5-Pad1): track 3.17 -> 6.35 mm
Changed lines of the file:
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@@
     (thickness 1.6)
     (drawings 7)
-    (tracks 125)
+    (tracks 143)
     (zones 0)
     (modules 18)
@@
     )
   )
-  (module Power_Supply:HLK-PM01 locked (layer F.Cu)
-    (at 172.72 105.41 75)
-    (fp_text reference U2 (at -17.78 -9.398 165) (layer F.SilkS)
-      (effects (font (size 0.762 0.762) (thickness 0.127)))
-    )
-    (fp_text value HLK-PM03 (at 0 11 75) (layer F.Fab)
-      (effects (font (size 0.762 0.762) (thickness 0.127)))
-    )
-    (fp_line (start 17 -10) (end -17 -10) (layer F.SilkS) (width 0.127))
-    (fp_line (start -17 10) (end 17 10) (layer F.SilkS) (width 0.127))
-    (fp_line (start -17 -10) (end -17 10) (layer F.SilkS) (width 0.127))
-    (fp_line (start 17 10) (end 17 -10) (layer F.SilkS) (width 0.127))
-    (pad 4 thru_hole circle (at 14.7 7.7 75) (size 2.2 2.2) (drill 1.25) (layers *.Cu *.Mask)
-      (net 26 "Net-(D1-Pad1)"))
-    (pad 3 thru_hole circle (at 14.7 -7.7 75) (size 2.2 2.2) (drill 1.25) (layers *.Cu *.Mask)
-      (net 1 GND))
-    (pad 2 thru_hole circle (at -14.7 2.5 75) (size 2.2 2.2) (drill 1.25) (layers *.Cu *.Mask)
-      (net 23 "Net-(J1-Pad1)"))
-    (pad 1 thru_hole circle (at -14.7 -2.5 75) (size 2.2 2.2) (drill 1.25) (layers *.Cu *.Mask)
-      (net 25 "Net-(BR1-Pad4)"))
-    (model C:/Engineering/KiCAD_Libraries/3D/Power_Supplies/AC_DC_Converters/VRML/HLK-PM01.wrl
-      (at (xyz 0 0 0))
-      (scale (xyz 1 1 1))
-      (rotate (xyz 0 0 0))
-    )
-  )
   (module wemos-d1-mini:wemos-d1-mini-embedded (layer F.Cu)
     (at 146.825 71.565 90)
@@
     )
   )
+  (module Power_Supply:HLK-PM01 locked (layer F.Cu)
+    (at 172.72 105.41 75)
+    (fp_text reference U2 (at -17.78 -9.398 165) (layer F.SilkS)
+      (effects (font (size 0.762 0.762) (thickness 0.127)))
+    )
+    (fp_text value HLK-PM03 (at 0 11 75) (layer F.Fab)
+      (effects (font (size 0.762 0.762) (thickness 0.127)))
+    )
+    (fp_line (start 17 -10) (end -17 -10) (layer F.SilkS) (width 0.127))
+    (fp_line (start -17 10) (end 17 10) (layer F.SilkS) (width 0.127))
+    (fp_line (start -17 -10) (end -17 10) (layer F.SilkS) (width 0.127))
+    (fp_line (start 17 10) (end 17 -10) (layer F.SilkS) (width 0.127))
+    (pad 4 thru_hole circle (at 14.7 7.7 75) (size 2.2 2.2) (drill 1.25) (layers *.Cu *.Mask)
+      (net 26 "Net-(D1-Pad1)"))
+    (pad 3 thru_hole circle (at 14.7 -7.7 75) (size 2.2 2.2) (drill 1.25) (layers *.Cu *.Mask)
+      (net 1 GND))
+    (pad 2 thru_hole circle (at -14.7 2.5 75) (size 2.2 2.2) (drill 1.25) (layers *.Cu *.Mask)
+      (net 23 "Net-(J1-Pad1)"))
+    (pad 1 thru_hole circle (at -14.7 -2.5 75) (size 2.2 2.2) (drill 1.25) (layers *.Cu *.Mask)
+      (net 25 "Net-(BR1-Pad4)"))
+    (model C:/Engineering/KiCAD_Libraries/3D/Power_Supplies/AC_DC_Converters/VRML/HLK-PM01.wrl
+      (at (xyz 0 0 0))
+      (scale (xyz 1 1 1))
+      (rotate (xyz 0 0 0))
+    )
+  )
   (gr_circle (center 146.825 98.565) (end 188.325 98.565) (layer Edge.Cuts) (width 0.2))
   (gr_circle (center 105.325 98.565) (end 112.825 98.565) (layer Edge.Cuts) (width 0.2))
@@
   (segment (start 154.305 85.09) (end 158.75 85.09) (width 0.25) (layer F.Cu) (net 2))
   (segment (start 130.175 105.41) (end 130.175 108.585) (width 2) (layer F.Cu) (net 3))
+  (segment (start 130.175 108.585) (end 130.175 105.41) (width 2) (layer B.Cu) (net 3))
   (segment (start 131.445 127) (end 131.445 118.745) (width 0.25) (layer F.Cu) (net 4))
   (segment (start 141.605 93.98) (end 140.97 93.345) (width 0.25) (layer F.Cu) (net 4))
@@
   (segment (start 118.11 107.95) (end 123.745 113.585) (width 2) (layer F.Cu) (net 22))
   (segment (start 130.175 113.585) (end 126.365 117.395) (width 2) (layer F.Cu) (net 22))
+  (segment (start 123.745 113.585) (end 130.175 113.585) (width 2) (layer B.Cu) (net 22))
+  (segment (start 118.11 107.95) (end 123.745 113.585) (width 2) (layer B.Cu) (net 22))
+  (segment (start 126.365 117.395) (end 126.365 127) (width 2) (layer B.Cu) (net 22))
+  (segment (start 130.175 113.585) (end 126.365 117.395) (width 2) (layer B.Cu) (net 22))
   (segment (start 121.285 95.885) (end 124.46 92.71) (width 2) (layer F.Cu) (net 23))
   (segment (start 124.46 92.71) (end 130.175 92.71) (width 2) (layer F.Cu) (net 23))
@@
   (segment (start 160.02 116.205) (end 167.279018 116.205) (width 1) (layer F.Cu) (net 23))
   (segment (start 144.145 107.315) (end 151.13 107.315) (width 1) (layer F.Cu) (net 23))
+  (segment (start 121.285 95.885) (end 124.46 92.71) (width 2) (layer B.Cu) (net 23))
+  (segment (start 124.46 92.71) (end 130.175 92.71) (width 2) (layer B.Cu) (net 23))
+  (segment (start 132.715 102.87) (end 135.255 105.41) (width 2) (layer B.Cu) (net 23))
+  (segment (start 130.175 92.71) (end 132.715 95.25) (width 2) (layer B.Cu) (net 23))
+  (segment (start 132.715 95.25) (end 132.715 102.87) (width 2) (layer B.Cu) (net 23))
+  (segment (start 135.255 105.41) (end 135.255 112.395) (width 2) (layer B.Cu) (net 23))
+  (segment (start 135.255 112.395) (end 128.905 118.745) (width 2) (layer B.Cu) (net 23))
+  (segment (start 128.905 118.745) (end 128.905 127) (width 2) (layer B.Cu) (net 23))
   (segment (start 132.715 128.905) (end 133.35 128.27) (width 0.25) (layer F.Cu) (net 24))
   (segment (start 124.46 128.27) (end 125.095 128.905) (width 0.25) (layer F.Cu) (net 24))
@@
   (segment (start 113.386528 110.410732) (end 113.386528 103.783472) (width 3) (layer F.Cu) (net 25))
   (segment (start 115.57 88.32532) (end 117.396936 86.498384) (width 3) (layer F.Cu) (net 25))
+  (segment (start 113.386528 110.410732) (end 114.517898 111.542102) (width 3) (layer B.Cu) (net 25))
+  (segment (start 115.57 101.6) (end 113.386528 103.783472) (width 3) (layer B.Cu) (net 25))
+  (segment (start 117.396936 86.498384) (end 115.57 88.32532) (width 3) (layer B.Cu) (net 25))
+  (segment (start 113.386528 103.783472) (end 113.386528 110.410732) (width 3) (layer B.Cu) (net 25))
+  (segment (start 115.57 88.32532) (end 115.57 101.6) (width 3) (layer B.Cu) (net 25))
   (segment (start 171.02 80.455) (end 171.12 80.555) (width 0.25) (layer F.Cu) (net 26))
   (segment (start 163.335 80.455) (end 171.02 80.455) (width 0.25) (layer F.Cu) (net 26))
@@
       )
     )
-  )
-  (zone (net 0) (net_name "") (layers F&B.Cu) (hatch edge 0.508)
-    (connect_pads (clearance 0.508))
-    (min_thickness 0.254)
-    (keepout (tracks not_allowed) (vias not_allowed) (copperpour allowed))
-    (fill (arc_segments 16) (thermal_gap 0.508) (thermal_bridge_width 0.508))
-    (polygon
-      (pts
-        (xy 112.395 85.09) (xy 120.015 81.915) (xy 123.19 88.9) (xy 141.605 88.9) (xy 145.415 92.71)
-        (xy 145.415 105.41) (xy 151.765 105.41) (xy 160.655 114.3) (xy 168.91 114.3) (xy 173.99 120.015)
-        (xy 173.355 121.92) (xy 171.45 122.555) (xy 169.545 121.92) (xy 168.275 120.65) (xy 155.575 120.65)
-        (xy 145.415 120.65) (xy 141.605 123.19) (xy 141.605 131.445) (xy 118.745 131.445) (xy 109.855 120.015)
-        (xy 109.855 102.235) (xy 112.395 99.695)
-      )
-    )
