File: ceiling-light-controller/circuits/ceiling-light-controller.sch (KiCad schematic (older format))
At the start: 18 parts, among them J1 Screw_Terminal_01x03, J2 Screw_Terminal_01x02, Q1 BT136-500, U1 LTV-817, U2 HLK-PM03, U3 MOC3021M, U4 WeMos_mini

Commit message: fixing submodule path once again
Parts:
- removed U2: HLK-PM03, Power_Supply:HLK-PM01, symbol Power_Supplies:HLK-PM03
- added U2: HLK-PM05, Power_Supply:HLK-PM05, symbol Power_Supplies:HLK-PM05
Changed lines of the file:
@@
 	2050 1700 1650 1700
-$Comp
-L Power_Supplies:HLK-PM03 U2
-U 1 1 5CE9C5F6
-P 2350 1750
-F 0 "U2" H 2350 1992 40  0000 C CNN
-F 1 "HLK-PM03" H 2350 1916 40  0000 C CNN
-F 2 "Power_Supply:HLK-PM01" H 1450 3100 60  0001 C CNN
-F 3 "" H 1450 3100 60  0000 C CNN
-	1    2350 1750
-	1    0    0    -1
-$EndComp
 $Comp
 L wemos_mini:WeMos_mini U4
@@
 Wire Wire Line
 	1650 1050 1550 1050
+$Comp
+L Power_Supplies:HLK-PM05 U2
+U 1 1 5CEC553E
+P 2350 1750
+F 0 "U2" H 2350 1992 40  0000 C CNN
+F 1 "HLK-PM05" H 2350 1916 40  0000 C CNN
+F 2 "Power_Supply:HLK-PM05" H 1450 3100 60  0001 C CNN
+F 3 "" H 1450 3100 60  0000 C CNN
+	1    2350 1750
+	1    0    0    -1
+$EndComp
 $EndSCHEMATC
