File: mains-light-controller/circuits/mains-light-controller.sch (KiCad schematic (older format))
At the start: 18 parts, among them J1 Screw_Terminal_01x03, J2 Screw_Terminal_01x02, Q1 BT136-500, U1 LTV-817, U2 HLK-PM05, U3 MOC3021M, U4 WeMos_mini

Commit message: improved schematic layout view; missing new PCB layout
Parts:
- added R8: 10K, Resistor_THT:R_Axial_DIN0207_L6.3mm_D2.5mm_P7.62mm_Horizontal, symbol Device:R
- added SW1: SW_Push, Button_Switch_THT:SW_PUSH_6mm, symbol Switch:SW_Push
- C1: value 1µf -> 1µF
- C5: value 100nf -> 100NF
- R1: value 390k -> 390K
- R2: value 10k -> 10K; footprint Resistor_THT:R_Axial_DIN0309_L9.0mm_D3.2mm_P12.70mm_Horizontal -> Resistor_THT:R_Axial_DIN0207_L6.3mm_D2.5mm_P7.62mm_Horizontal
- R3: value 10k -> 10K
- R4: value 100 -> 100R
- R5: value 330 -> 33R; footprint Resistor_THT:R_Axial_DIN0309_L9.0mm_D3.2mm_P12.70mm_Horizontal -> Resistor_THT:R_Axial_DIN0207_L6.3mm_D2.5mm_P7.62mm_Horizontal
- R6: value 10000 -> 10K; footprint Resistor_THT:R_Axial_DIN0309_L9.0mm_D3.2mm_P12.70mm_Horizontal -> Resistor_THT:R_Axial_DIN0207_L6.3mm_D2.5mm_P7.62mm_Horizontal
- U2: footprint Power_Supply:HLK-PM05 -> Power_Supply:HLK-PM01
Connections:
- net labels added: +3V3, +5V, A0, D0, D1, D2, D3, D4, D5, D6, D7, D8, L_OUT, M1_IN, M2_IN, N_MAIN, RST, RX, TX
- wire segments 62 -> 80
Other:
- note added: "HUMIDITY SENSE"
- note added: "L"
- note added: "LIGHT SENSE"
- note added: "M1"
- note added: "M2"
- note added: "MAINS AC-DV 5V CONVERTER"
- note added: "MAINS INPUT"
- note added: "MAINS OUTPUT"
- note added: "MAINS POWER SENSE"
- note added: "MAINS POWER SWITCHING"
- note added: "MCU"
- note added: "N"
- note added: "RGB LED STATUS"
- note added: "SWITCH BUTTON"
- note added: "TEMPERATURE SENSE"
- moved on the sheet: BR1, C1, D1, J1, J2, Q1, R1, R3, R4, R5, R6, R7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

Commit message: Schematic changes; PCB component placement, no traces
Other:
- note added: "3.3V supply lowers interface logics"
- note added: "MAIN MCU\n"
- note added: "NOT YET AVAILABLE\n"
- note removed: "MCU"
- moved on the sheet: BR1, C1, D1, R1, R2, R8, SW1, U1, U2, U4

Commit message: new PCB layout and traces for mains light controller
Parts:
- added F1: Fuse, Fuse_Holders_and_Fuses:Fuseholder5x20_horiz_open_lateral_Type-II, symbol Device:Fuse
- R1, R3: footprint Resistor_THT:R_Axial_DIN0309_L9.0mm_D3.2mm_P12.70mm_Horizontal -> Resistor_SMD:R_1206_3216Metric_Pad1.42x1.75mm_HandSolder
- R2, R5, R6, R8: footprint Resistor_THT:R_Axial_DIN0207_L6.3mm_D2.5mm_P7.62mm_Horizontal -> Resistor_SMD:R_1206_3216Metric_Pad1.42x1.75mm_HandSolder
- R4: footprint Resistor_THT:R_Axial_DIN0309_L9.0mm_D3.2mm_P12.70mm_Horizontal -> Resistor_SMD:R_2010_5025Metric_Pad1.52x2.65mm_HandSolder
- R7: footprint OptoDevice:R_LDR_10x8.5mm_P7.6mm_Vertical -> OptoDevice:R_LDR_5.0x4.1mm_P3mm_Vertical
- U4: footprint wemos-d1-mini:wemos-d1-mini-embedded -> wemos-d1-mini:wemos-d1-mini-connectors-only
Connections:
- wire segments 80 -> 81
Other:
- moved on the sheet: Q1, R3, R4, R5, SW1, U3, U4

Commit message: load switching with FL5150
Parts:
- removed C5: 100NF, Capacitor_THT:C_Disc_D5.1mm_W3.2mm_P5.00mm, symbol Device:C
- removed Q1: BT136-500, slimc:TO-220-3_Vertical_Triode_Heatsink, symbol Triac_Thyristor:BT136-500
- removed R3: 10K, Resistor_SMD:R_1206_3216Metric_Pad1.42x1.75mm_HandSolder, symbol Device:R
- removed R4: 100R, Resistor_SMD:R_2010_5025Metric_Pad1.52x2.65mm_HandSolder, symbol Device:R
- removed R5: 33R, Resistor_SMD:R_1206_3216Metric_Pad1.42x1.75mm_HandSolder, symbol Device:R
- removed U3: MOC3021M, Package_DIP:DIP-6_W7.62mm, symbol Relay_SolidState:MOC3021M
- added C? (x2): 22nF, symbol Device:C_Small
- added C? (x2): 100nF, symbol Device:C_Small
- added D?: 1N4007, Diode_THT:D_DO-41_SOD81_P10.16mm_Horizontal, symbol Diode:1N4007
- added Q? (x2): IRF840, Package_TO_SOT_THT:TO-220-3_Vertical, symbol Transistor_FET:IRF740
- added Q?: KSP44, Package_TO_SOT_THT:TO-39-3, symbol Transistor_BJT:2N2219
- added R? (x3): 2M, Resistor_SMD:R_1206_3216Metric_Pad1.42x1.75mm_HandSolder, symbol Device:R
- added R?: 1K, Resistor_SMD:R_1206_3216Metric_Pad1.42x1.75mm_HandSolder, symbol Device:R
- added R?: 33K, Resistor_SMD:R_1206_3216Metric_Pad1.42x1.75mm_HandSolder, symbol Device:R
- added R?: 330K, Resistor_SMD:R_1206_3216Metric_Pad1.42x1.75mm_HandSolder, symbol Device:R
- added U?: FL5150MX, symbol AC_Drivers:FL5150MX
- added U?: AMS1117-5.0, Package_TO_SOT_SMD:SOT-223-3_TabPin2, symbol Regulator_Linear:AMS1117-5.0
Connections:
- net labels added: +12V
- wire segments 81 -> 119
Other:
- note added: "5VDC CONVERTER"
- note added: "MAINS ACDC 12V CONVERTER"
- note removed: "MAINS AC-DV 5V CONVERTER"
- moved on the sheet: R6, R7, R8, SW1, U2, U4

Commit message: mlc dimmerable edition in own directory
Parts:
- removed C? (x2): 22nF, symbol Device:C_Small
- removed C? (x2): 100nF, symbol Device:C_Small
- removed D?: 1N4007, Diode_THT:D_DO-41_SOD81_P10.16mm_Horizontal, symbol Diode:1N4007
- removed Q? (x2): IRF840, Package_TO_SOT_THT:TO-220-3_Vertical, symbol Transistor_FET:IRF740
- removed Q?: KSP44, Package_TO_SOT_THT:TO-39-3, symbol Transistor_BJT:2N2219
- removed R? (x3): 2M, Resistor_SMD:R_1206_3216Metric_Pad1.42x1.75mm_HandSolder, symbol Device:R
- removed R?: 1K, Resistor_SMD:R_1206_3216Metric_Pad1.42x1.75mm_HandSolder, symbol Device:R
- removed R?: 33K, Resistor_SMD:R_1206_3216Metric_Pad1.42x1.75mm_HandSolder, symbol Device:R
- removed R?: 330K, Resistor_SMD:R_1206_3216Metric_Pad1.42x1.75mm_HandSolder, symbol Device:R
- removed U?: FL5150MX, symbol AC_Drivers:FL5150MX
- removed U?: AMS1117-5.0, Package_TO_SOT_SMD:SOT-223-3_TabPin2, symbol Regulator_Linear:AMS1117-5.0
- added C5: 100NF, Capacitor_THT:C_Disc_D5.1mm_W3.2mm_P5.00mm, symbol Device:C
- added Q1: BT136-500, slimc:TO-220-3_Vertical_Triode_Heatsink, symbol Triac_Thyristor:BT136-500
- added R3: 10K, Resistor_SMD:R_1206_3216Metric_Pad1.42x1.75mm_HandSolder, symbol Device:R
- added R4: 100R, Resistor_SMD:R_2010_5025Metric_Pad1.52x2.65mm_HandSolder, symbol Device:R
- added R5: 33R, Resistor_SMD:R_1206_3216Metric_Pad1.42x1.75mm_HandSolder, symbol Device:R
- added U3: MOC3021M, Package_DIP:DIP-6_W7.62mm, symbol Relay_SolidState:MOC3021M
Connections:
- net labels removed: +12V
- wire segments 119 -> 81
Other:
- note added: "MAINS AC-DV 5V CONVERTER"
- note removed: "5VDC CONVERTER"
- note removed: "HUMIDITY SENSE"
- note removed: "MAINS ACDC 12V CONVERTER"
- note removed: "NOT YET AVAILABLE\n"
- note removed: "TEMPERATURE SENSE"
- moved on the sheet: R6, R7, R8, SW1, U2, U4
