File: ceiling-light/circuits/undimmable/ceiling-light.kicad_pcb (KiCad board)
At the start: 2 copper layers, 100 x 100 mm, 21 parts, among them J1 Screw_Terminal_01x03, J2 Screw_Terminal_01x02, Q1 BT136-500, SW1 SW_Push, U1 LTV-817, U2 HLK-PM05, U3 MOC3021M, U4 WeMos_mini

Commit message: work on dimmable circuit and git submodules
Parts:
- added C2: 0.1µF, Capacitor_THT:C_Disc_D5.1mm_W3.2mm_P5.00mm, F.Cu at (190.8, 73.1)
- added C3: 0.1µF, Capacitor_THT:C_Disc_D5.1mm_W3.2mm_P5.00mm, F.Cu at (193.0, 76.9)
- added J3: Conn_01x04, Connector_PinHeader_2.54mm:PinHeader_1x04_P2.54mm_Vertical, F.Cu at (191.6, 61.8)
- added J4: Conn_01x04, Connector_PinHeader_2.54mm:PinHeader_1x04_P2.54mm_Vertical, F.Cu at (175.9, 77.8)
- added J5: Conn_01x04, Connector_PinHeader_2.54mm:PinHeader_1x04_P2.54mm_Vertical, F.Cu at (187.8, 29.2)
- added U5: ESP32-WROOM-32D, RF_Module:ESP32-WROOM-32, F.Cu at (168.0, 39.2)
- C5: value 100NF -> 100nF
- Q1: footprint slimc:TO-220-3_Vertical_Triode_Heatsink -> Package_TO_SOT_THT:TO-220-3_Horizontal_TabUp
- U4: value WeMos_mini -> TMP36xS; footprint wemos-d1-mini:wemos-d1-mini-connectors-only -> Package_SO:SOIC-8_3.9x4.9mm_P1.27mm
- moved D1 152.2 mm to (177.9, 90.1), turned to 0 degrees
- moved R8 148.2 mm to (195.9, 69.3), turned to 0 degrees
- moved R2 147.4 mm to (200.8, 69.3), turned to 0 degrees
- moved U3 140.9 mm to (194.5, 61.6), turned to 0 degrees
- moved R1 136.6 mm to (199.4, 71.6), turned to 0 degrees
- moved R4 134.2 mm to (185.0, 85.7)
- moved R3 132.9 mm to (184.1, 88.4)
- moved C1 129.4 mm to (188.1, 89.6), turned to 0 degrees
- moved Q1 129.4 mm to (166.3, 69.2), turned to 0 degrees
- moved J2 127.0 mm to (184.1, 80.0), turned to 0 degrees
- moved F1 123.4 mm to (169.0, 61.4)
- moved C5 122.4 mm to (175.2, 94.8), turned to 0 degrees
- moved R6 115.3 mm to (201.6, 73.9), turned to 0 degrees
- moved R5 113.8 mm to (156.9, 98.1), turned to 0 degrees
- moved SW1 112.5 mm to (146.4, 93.1), turned to 0 degrees
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Connections:
- C1 pad 1: D1 -> Net-(C1-Pad1)
- D1 pad 4: D4 -> Net-(D1-Pad4)
- R2 pad 1: D1 -> Net-(C1-Pad1)
- R5 pad 2: D2 -> Net-(R5-Pad2)
- R6 pad 1: A0 -> Net-(R6-Pad1)
- R7 pad 2: A0 -> Net-(R6-Pad1)
- R8 pad 2: D3 -> Net-(R8-Pad2)
- SW1 pad 1: D3 -> Net-(R8-Pad2)
- U1 pad 4: D1 -> Net-(C1-Pad1)
- U2 pad 4: +5V -> +3V3
- U4 pad 1: +5V -> Net-(U4-Pad1)
- U4 pad 2: GND -> (no net)
- U4 pad 3: D4 -> (no net)
- U4 pad 4: D3 -> GND
- U4 pad 5: D2 -> +3V3
- U4 pad 6: D1 -> (no net)
- U4 pad 7: RX -> (no net)
- U4 pad 8: TX -> +3V3
Routing:
- net M2_IN: track 204.0 -> 0.00 mm
- net +3V3: track 134.2 -> 0.00 mm
- net N_MAIN: track 76.0 -> 0.00 mm
- net +5V: track 59.0 -> 0.00 mm
- net Net-(F1-Pad2): track 52.9 -> 0.00 mm
- net D4: track 43.1 -> 0.00 mm
- net L_OUT: track 41.8 -> 0.00 mm
- net A0: track 37.7 -> 0.00 mm
- net D3: track 35.6 -> 0.00 mm
- net D1: track 34.8 -> 0.00 mm
- net D2: track 22.8 -> 0.00 mm
- net M1_IN: track 21.9 -> 0.00 mm
- net Net-(Q1-Pad3): track 17.4 -> 0.00 mm
- net Net-(BR1-Pad1): track 11.3 -> 0.00 mm
- net Net-(BR1-Pad2): track 6.24 -> 0.00 mm
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- removed copper zone on B.Cu, net GND
- removed copper zone on F.Cu, net GND
