File: ceiling-light/circuits/undimmable/ceiling-light.sch (KiCad schematic (older format))
At the start: 22 parts, among them J1 Screw_Terminal_01x03, J2 Screw_Terminal_01x02, Q1 BT136-500, SW1 SW_Push, U1 LTV-817, U2 HLK-PM05, U3 MOC3021M, U4 WeMos_mini

Commit message: work on dimmable circuit and git submodules
Parts:
- removed U4: WeMos_mini, wemos-d1-mini:wemos-d1-mini-connectors-only, symbol wemos_mini:WeMos_mini
- added C2, C3: 0.1µF, Capacitor_THT:C_Disc_D5.1mm_W3.2mm_P5.00mm, symbol Device:C
- added J3, J4: Conn_01x04, Connector_PinHeader_2.54mm:PinHeader_1x04_P2.54mm_Vertical, symbol Connector_Generic:Conn_01x04
- added J?: Conn_01x05, symbol Connector_Generic:Conn_01x05
- added U4: TMP36xS, Package_SO:SOIC-8_3.9x4.9mm_P1.27mm, symbol Sensor_Temperature:TMP36xS
- C5: value 100NF -> 100nF
- Q1: footprint slimc:TO-220-3_Vertical_Triode_Heatsink -> Package_TO_SOT_THT:TO-220-3_Horizontal_TabUp
- gave numbers to parts that had none: 1
Connections:
- net labels added: RXD, SENSE_VP, SENSOR_VN, SENSOR_VP, TXD
- net labels removed: +5V, A0, D0, D1, D2, D3, D4, D5, D6, D7, D8, RX, TX
- wire segments 83 -> 93
Other:
- note added: "MAIN MCU"
- note added: "MAINS AC-DV 3V3 CONVERTER"
- note added: "MAINS SCREW TERMINALS"
- note added: "PIN HEADERS"
- note added: "PROGRAMMING HEADER"
- note added: "PWR"
- note added: "SW"
- note added: "TEMPERATURE SENSOR"
- note removed: "3.3V supply lowers interface logics"
- note removed: "L"
- note removed: "M1"
- note removed: "M2"
- note removed: "MAIN MCU\n"
- note removed: "MAINS AC-DV 5V CONVERTER"
- note removed: "MAINS INPUT"
- note removed: "MAINS OUTPUT"
- note removed: "N"
- moved on the sheet: BR1, C1, C5, D1, F1, J1, J2, Q1, R1, R2, R3, R4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
