File: ceiling-light/circuits/dimmable/ceiling-light-dimmable.sch (KiCad schematic (older format))
At the start: 31 parts, among them J1 Screw_Terminal_01x03, J2 Screw_Terminal_01x02, SW1 SW_Push, U1 LTV-817, U2 HLK-PM05, U4 WeMos_mini

Commit message: work on dimmable circuit and git submodules
Parts:
- removed BR1: DB107-BP, DB107-BP:DIP825W56P510L828H330Q4N, symbol DB107-BP:DB107-BP
- removed C?: 100nF, symbol Device:C_Small
- removed R8: 10K, Resistor_SMD:R_1206_3216Metric_Pad1.42x1.75mm_HandSolder, symbol Device:R
- removed R?: 2M, Resistor_SMD:R_1206_3216Metric_Pad1.42x1.75mm_HandSolder, symbol Device:R
- removed U4: WeMos_mini, wemos-d1-mini:wemos-d1-mini-connectors-only, symbol wemos_mini:WeMos_mini
- removed U?: FL5150MX, symbol AC_Drivers:FL5150MX
- removed U?: AMS1117-5.0, Package_TO_SOT_SMD:SOT-223-3_TabPin2, symbol Regulator_Linear:AMS1117-5.0
- added BR?: DB107-BP, DIP825W56P510L828H330Q4N, symbol Diode_Bridge:DB107-BP
- added C5, C6: 0.1µF, symbol Device:C_Small
- added J3: Conn_01x07, Connector_PinSocket_2.54mm:PinSocket_1x07_P2.54mm_Vertical, symbol Connector_Generic:Conn_01x07
- added J4, J5: Conn_01x01, Connector_PinSocket_2.54mm:PinSocket_1x01_P2.54mm_Vertical, symbol Connector_Generic:Conn_01x01
- added R12: 2M, Resistor_SMD:R_1206_3216Metric_Pad1.42x1.75mm_HandSolder, symbol Device:R
- added SW2, SW3: SW_Push, Button_Switch_SMD:SW_SPST_B3S-1000, symbol Switch:SW_Push
- added U3: AMS1117-3.3, Package_TO_SOT_SMD:SOT-223-3_TabPin2, symbol Regulator_Linear:AMS1117-3.3
- added U4: FL51xxMX, slimc:FL51xxMX, symbol AC_Drivers:FL51xxMX
- added U5: TMP36xS, Package_SO:SOIC-8_3.9x4.9mm_P1.27mm, symbol Sensor_Temperature:TMP36xS
- added U6: ESP32-WROOM-32D, RF_Module:ESP32-WROOM-32, symbol RF_Module:ESP32-WROOM-32D
- R5: renamed from R?; value 33K -> 330K
- R6: value 10K -> 6K8
- R9: renamed from R?; value 330K -> 33K
- gave numbers to parts that had none: 10
Connections:
- net labels added: DIMCN, DIM_MODE, ESP_FLASH, ESP_RX, ESP_TX, LIGHT_SENSE, MAINS_SENSE, STATUS_LED, TEMP_SENSE
- net labels removed: +12V, A0, D0, D1, D2, D3, D4, D5, D6, D7, D8, RST, RX, TX
- wire segments 119 -> 141
- no-connect marks 0 -> 1
Other:
- note added: "3V3 DC CONVERTER"
- note added: "5V ACDC CONVERTER"
- note added: "CONSTANT"
- note added: "DIM CONTROL DAC"
- note added: "FTDI 5V\n"
- note added: "FTDI GND"
- note added: "FTDI PROGRAMMING HEADER"
- note added: "FTDI RST"
- note added: "FTDI RXD"
- note added: "FTDI TXD"
- note added: "FTDI/PWR 3V3"
- note added: "FTDI/PWR GND"
- note added: "LIGHT SENSER"
- note added: "LIVE LOAD"
- note added: "NEUTRAL"
- note added: "RGB STATUS LED"
- note added: "SWITCH"
- note added: "TEMPERATURE SENSOR"
- note removed: "3.3V supply lowers interface logics"
- note removed: "5VDC CONVERTER"
- note removed: "HUMIDITY SENSE"
- note removed: "L"
- note removed: "LIGHT SENSE"
- note removed: "M1"
- note removed: "M2"
- note removed: "MAIN MCU\n"
- note removed: "MAINS ACDC 12V CONVERTER"
- note removed: "N"
- note removed: "NOT YET AVAILABLE\n"
- note removed: "SWITCH BUTTON"
- note removed: "TEMPERATURE SENSE"
- moved on the sheet: C1, C2, C3, C4, D1, D2, F1, J1, J2, Q2, Q3, Q4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

Commit message: git submodule fixing
Parts:
- BR1: renamed from BR?; footprint DIP825W56P510L828H330Q4N -> Diode_THT:DB107-BP
- C2: footprint (none) -> Capacitor_THT:C_Radial_D10.0mm_H12.5mm_P5.00mm
- C3, C4, C5, C6: footprint (none) -> Capacitor_THT:C_Radial_D4.0mm_H5.0mm_P1.50mm
- U4: footprint slimc:FL51xxMX -> AC_Drivers:FL51xxMX
Changed lines of the file:
@@
 F 0 "C2" V 2921 1400 50  0000 C CNN
 F 1 "22nF" V 3012 1400 50  0000 C CNN
-F 2 "" H 3150 1400 50  0001 C CNN
+F 2 "Capacitor_THT:C_Radial_D10.0mm_H12.5mm_P5.00mm" H 3150 1400 50  0001 C CNN
 F 3 "~" H 3150 1400 50  0001 C CNN
 	1    3150 1400
@@
 F 0 "C4" H 5758 1554 50  0000 R CNN
 F 1 "100nF" H 5758 1645 50  0000 R CNN
-F 2 "" H 5850 1600 50  0001 C CNN
+F 2 "Capacitor_THT:C_Radial_D4.0mm_H5.0mm_P1.50mm" H 5850 1600 50  0001 C CNN
 F 3 "~" H 5850 1600 50  0001 C CNN
 	1    5850 1600
@@
 F 0 "U4" H 4550 1925 50  0000 C CNN
 F 1 "FL51xxMX" H 4550 1834 50  0000 C CNN
-F 2 "slimc:FL51xxMX" H 4200 1900 50  0001 C CNN
+F 2 "AC_Drivers:FL51xxMX" H 4200 1900 50  0001 C CNN
 F 3 "" H 4200 1900 50  0001 C CNN
 	1    4550 1500
@@
 F 0 "C3" V 4400 2050 50  0000 R CNN
 F 1 "22nF" V 4300 2050 50  0000 R CNN
-F 2 "" H 4550 1950 50  0001 C CNN
+F 2 "Capacitor_THT:C_Radial_D4.0mm_H5.0mm_P1.50mm" H 4550 1950 50  0001 C CNN
 F 3 "~" H 4550 1950 50  0001 C CNN
 	1    4550 1950
@@
 F 0 "C5" H 800 5250 50  0000 R CNN
 F 1 "0.1µF" H 950 5150 50  0000 R CNN
-F 2 "" H 850 5450 50  0001 C CNN
+F 2 "Capacitor_THT:C_Radial_D4.0mm_H5.0mm_P1.50mm" H 850 5450 50  0001 C CNN
 F 3 "~" H 850 5450 50  0001 C CNN
 	1    850  5450
@@
 F 0 "C6" H 2900 5250 50  0000 R CNN
 F 1 "0.1µF" H 3000 5100 50  0000 R CNN
-F 2 "" H 3050 5200 50  0001 C CNN
+F 2 "Capacitor_THT:C_Radial_D4.0mm_H5.0mm_P1.50mm" H 3050 5200 50  0001 C CNN
 F 3 "~" H 3050 5200 50  0001 C CNN
 	1    3050 5200
@@
 $EndComp
 $Comp
-L Diode_Bridge:DB107-BP BR?
+L Diode_Bridge:DB107-BP BR1
 U 1 1 5D45626B
 P 3450 3450
-F 0 "BR?" H 3900 3715 50  0000 C CNN
+F 0 "BR1" H 3900 3715 50  0000 C CNN
 F 1 "DB107-BP" H 3900 3624 50  0000 C CNN
-F 2 "DIP825W56P510L828H330Q4N" H 4200 3550 50  0001 L CNN
+F 2 "Diode_THT:DB107-BP" H 4200 3550 50  0001 L CNN
 F 3 "http://www.mccsemi.com/up_pdf/DB101-DB107(DB-1).pdf" H 4200 3450 50  0001 L CNN
 F 4 "Bridge Rectifiers 1.0A 1000V" H 4200 3350 50  0001 L CNN "Description"

Commit message: submodule update and plot export
Parts:
- removed BR1: DB107-BP, Diode_THT:DB107-BP, symbol Diode_Bridge:DB107-BP
- removed U4: FL51xxMX, AC_Drivers:FL51xxMX, symbol AC_Drivers:FL51xxMX
- added BR1: DB107-BP, Diode_THT_slimc:DB107-BP, symbol Diode_Bridge_slimc:DB107-BP
- added U4: FL51xxMX, AC_Drivers_slimc:FL51xxMX, symbol AC_Drivers_slimc:FL51xxMX
Connections:
- wire segments 141 -> 146
Changed lines of the file:
@@
 Rev "v1.1.0"
 Comp "slimc"
-Comment1 ""
+Comment1 "Open Source Project"
 Comment2 "github.com/slimcdk/smart-home-modules"
-Comment3 "Open Source Project"
-Comment4 "Auther: Christian Skjerning"
+Comment3 "Smart Home Modules"
+Comment4 "Auther: Christian Skjerning | slimc"
 $EndDescr
 $Comp
@@
 Wire Wire Line
 	5100 1150 5150 1150
-$Comp
-L AC_Drivers:FL51xxMX U4
-U 1 1 5D558438
-P 4550 1500
-F 0 "U4" H 4550 1925 50  0000 C CNN
-F 1 "FL51xxMX" H 4550 1834 50  0000 C CNN
-F 2 "AC_Drivers:FL51xxMX" H 4200 1900 50  0001 C CNN
-F 3 "" H 4200 1900 50  0001 C CNN
-	1    4550 1500
-	-1   0    0    -1
-$EndComp
 Wire Wire Line
 	3050 1400 2950 1400
@@
 $EndComp
 Wire Wire Line
-	4100 1400 3750 1400
-Wire Wire Line
-	3750 1500 4100 1500
-Wire Wire Line
-	3750 1300 4100 1300
+	4100 1400 4050 1400
+Wire Wire Line
+	3750 1500 4050 1500
+Wire Wire Line
+	3750 1300 4050 1300
 Wire Wire Line
 	2950 900  3400 900
@@
 Connection ~ 3800 1600
 Wire Wire Line
-	3800 1600 4100 1600
+	3800 1600 4050 1600
 Wire Wire Line
 	4050 1950 4050 1700
@@
 LIGHT_SENSE
 Wire Wire Line
-	2450 3450 2950 3450
+	2450 3450 2550 3450
 NoConn ~ 3200 5200
 Wire Notes Line
@@
 $EndComp
 $Comp
-L Diode_Bridge:DB107-BP BR1
-U 1 1 5D45626B
-P 3450 3450
-F 0 "BR1" H 3900 3715 50  0000 C CNN
-F 1 "DB107-BP" H 3900 3624 50  0000 C CNN
-F 2 "Diode_THT:DB107-BP" H 4200 3550 50  0001 L CNN
-F 3 "http://www.mccsemi.com/up_pdf/DB101-DB107(DB-1).pdf" H 4200 3450 50  0001 L CNN
-F 4 "Bridge Rectifiers 1.0A 1000V" H 4200 3350 50  0001 L CNN "Description"
-F 5 "3.3" H 4200 3250 50  0001 L CNN "Height"
-F 6 "Micro Commercial Components (MCC)" H 4200 3150 50  0001 L CNN "Manufacturer_Name"
-F 7 "DB107-BP" H 4200 3050 50  0001 L CNN "Manufacturer_Part_Number"
-F 8 "833-DB107-BP" H 4200 2950 50  0001 L CNN "Mouser Part Number"
-F 9 "https://www.mouser.com/Search/Refine.aspx?Keyword=833-DB107-BP" H 4200 2850 50  0001 L CNN "Mouser Price/Stock"
-	1    3450 3450
-	1    0    0    -1
-$EndComp
+L AC_Drivers_slimc:FL51xxMX U4
+U 1 1 5D445EC1
+P 4500 1500
+F 0 "U4" H 4500 1925 50  0000 C CNN
+F 1 "FL51xxMX" H 4500 1834 50  0000 C CNN
+F 2 "AC_Drivers_slimc:FL51xxMX" H 4150 1900 50  0001 C CNN
+F 3 "" H 4150 1900 50  0001 C CNN
+	1    4500 1500
+	1    0    0    -1
+$EndComp
+Connection ~ 4050 1300
+Wire Wire Line
+	4050 1300 4100 1300
+Connection ~ 4050 1400
+Wire Wire Line
+	4050 1400 3750 1400
+Connection ~ 4050 1500
+Wire Wire Line
+	4050 1500 4100 1500
+Connection ~ 4050 1600
+Wire Wire Line
+	4050 1600 4100 1600
+Connection ~ 4050 1700
+$Comp
+L Diode_Bridge_slimc:DB107-BP BR1
+U 1 1 5D4584FE
+P 4350 3450
+F 0 "BR1" H 4800 3715 50  0000 C CNN
+F 1 "DB107-BP" H 4800 3624 50  0000 C CNN
+F 2 "Diode_THT_slimc:DB107-BP" H 5100 3550 50  0001 L CNN
+F 3 "http://www.mccsemi.com/up_pdf/DB101-DB107(DB-1).pdf" H 5100 3450 50  0001 L CNN
+F 4 "Bridge Rectifiers 1.0A 1000V" H 5100 3350 50  0001 L CNN "Description"
+F 5 "3.3" H 5100 3250 50  0001 L CNN "Height"
+F 6 "Micro Commercial Components (MCC)" H 5100 3150 50  0001 L CNN "Manufacturer_Name"
+F 7 "DB107-BP" H 5100 3050 50  0001 L CNN "Manufacturer_Part_Number"
+F 8 "833-DB107-BP" H 5100 2950 50  0001 L CNN "Mouser Part Number"
+F 9 "https://www.mouser.com/Search/Refine.aspx?Keyword=833-DB107-BP" H 5100 2850 50  0001 L CNN "Mouser Price/Stock"
+	1    4350 3450
+	-1   0    0    -1
+$EndComp
+Connection ~ 2550 3450
+Wire Wire Line
+	2550 3450 2950 3450
 $EndSCHEMATC

Commit message: symbol was misaligned
Parts:
- BR1: symbol Diode_Bridge_slimc:DB107-BP -> ceiling-light-dimmable-rescue:DB107-BP-Diode_Bridge_slimc
- U4: symbol AC_Drivers_slimc:FL51xxMX -> ceiling-light-dimmable-rescue:FL51xxMX-AC_Drivers_slimc
Connections:
- wire segments 146 -> 141
Other:
- moved on the sheet: U4
Changed lines of the file:
@@
 $EndComp
-Wire Wire Line
-	4100 1400 4050 1400
-Wire Wire Line
-	3750 1500 4050 1500
-Wire Wire Line
-	3750 1300 4050 1300
 Wire Wire Line
 	2950 900  3400 900
@@
 Connection ~ 3800 1600
 Wire Wire Line
-	3800 1600 4050 1600
-Wire Wire Line
 	4050 1950 4050 1700
 Wire Wire Line
@@
 Text Label 2950 3450 2    50   ~ 0
 LIGHT_SENSE
-Wire Wire Line
-	2450 3450 2550 3450
 NoConn ~ 3200 5200
 Wire Notes Line
@@
 $EndComp
 $Comp
-L AC_Drivers_slimc:FL51xxMX U4
+L ceiling-light-dimmable-rescue:FL51xxMX-AC_Drivers_slimc U4
 U 1 1 5D445EC1
-P 4500 1500
-F 0 "U4" H 4500 1925 50  0000 C CNN
-F 1 "FL51xxMX" H 4500 1834 50  0000 C CNN
-F 2 "AC_Drivers_slimc:FL51xxMX" H 4150 1900 50  0001 C CNN
-F 3 "" H 4150 1900 50  0001 C CNN
-	1    4500 1500
-	1    0    0    -1
-$EndComp
-Connection ~ 4050 1300
-Wire Wire Line
-	4050 1300 4100 1300
-Connection ~ 4050 1400
-Wire Wire Line
-	4050 1400 3750 1400
-Connection ~ 4050 1500
-Wire Wire Line
-	4050 1500 4100 1500
-Connection ~ 4050 1600
-Wire Wire Line
-	4050 1600 4100 1600
-Connection ~ 4050 1700
-$Comp
-L Diode_Bridge_slimc:DB107-BP BR1
+P 4550 1500
+F 0 "U4" H 4550 1925 50  0000 C CNN
+F 1 "FL51xxMX" H 4550 1834 50  0000 C CNN
+F 2 "AC_Drivers_slimc:FL51xxMX" H 4200 1900 50  0001 C CNN
+F 3 "" H 4200 1900 50  0001 C CNN
+	1    4550 1500
+	1    0    0    -1
+$EndComp
+$Comp
+L ceiling-light-dimmable-rescue:DB107-BP-Diode_Bridge_slimc BR1
 U 1 1 5D4584FE
 P 4350 3450
@@
 	-1   0    0    -1
 $EndComp
-Connection ~ 2550 3450
-Wire Wire Line
-	2550 3450 2950 3450
+Wire Wire Line
+	2450 3450 2950 3450
+Wire Wire Line
+	3750 1300 4100 1300
+Wire Wire Line
+	3750 1400 4100 1400
+Wire Wire Line
+	3750 1500 4100 1500
+Wire Wire Line
+	3800 1600 4100 1600
 $EndSCHEMATC

Commit message: work on dimmable schematic
Parts:
- removed C1: 1µF, Capacitor_THT:CP_Radial_D4.0mm_P1.50mm, symbol Device:CP
- removed J3: Conn_01x07, Connector_PinSocket_2.54mm:PinSocket_1x07_P2.54mm_Vertical, symbol Connector_Generic:Conn_01x07
- removed J4, J5: Conn_01x01, Connector_PinSocket_2.54mm:PinSocket_1x01_P2.54mm_Vertical, symbol Connector_Generic:Conn_01x01
- removed SW3: SW_Push, Button_Switch_SMD:SW_SPST_B3S-1000, symbol Switch:SW_Push
- added J3: Conn_01x08, symbol Connector_Generic:Conn_01x08
- BR1: symbol ceiling-light-dimmable-rescue:DB107-BP-Diode_Bridge_slimc -> ceiling-light-dimmable-rescue:DB107-BP-Diode_Bridge_slimc-ceiling-light-dimmable-rescue
- U4: symbol ceiling-light-dimmable-rescue:FL51xxMX-AC_Drivers_slimc -> ceiling-light-dimmable-rescue:FL51xxMX-AC_Drivers_slimc-ceiling-light-dimmable-rescue
Connections:
- net +3V3: now also J3.4 (Pin_4)
- net +5V: now also U4.3 (VDD), J3.3 (Pin_3); no longer U4.8 (OCSen2)
- net DIMCN: now also U4.2 (DIMCN), U6.10 (IO25); no longer U4.9 (DRVG)
- net DIM_MODE: now also U4.4 (DM); no longer U4.7 (LPM)
- net GND: now also U4.5 (GND), J3.1 (Pin_1), J3.2 (Pin_2); no longer U4.6 (VS)
- net at R11.1: now also U4.9 (DRVG); no longer U4.2 (DIMCN)
- net at R10.1: now also U4.10 (OCSen1); no longer U4.1 (ZCMon)
- net at C3.1, Q4.1 (E): now also U4.6 (VS); no longer U4.5 (GND)
- net at Q4.2 (B), R5.1: now also U4.7 (LPM); no longer U4.4 (DM)
- net at R13.2: now also U4.1 (ZCMon); no longer U4.10 (OCSen1)
- net at R12.1: now also U4.8 (OCSen2); no longer U4.3 (VDD)
- net ESP_EN: now reaches SW2.2, U6.3 (EN)
- net ESP_EN: now also J3.7 (Pin_7)
- net ESP_FLASH renamed ESP_GPIO0
- net ESP_GPIO0: now also J3.8 (Pin_8)
- net ESP_RX renamed ESP_RXD0
- net ESP_RXD0: now also J3.6 (Pin_6)
- net ESP_TX renamed ESP_TXD0
- net ESP_TXD0: now also J3.5 (Pin_5)
- net MAINS_SENSE renamed SW_SENSE
- no-connect marks 1 -> 24
Other:
- note added: "3V3 PWR"
- note added: "5V PWR"
- note added: "ESP32-WROOM-32D MCU"
- note added: "FTDI DTR -> ESP GPIO0"
- note added: "FTDI RTS -> ESP EN"
- note added: "FTDI RXD -> ESP TXD"
- note added: "FTDI TXD -> ESP RXD"
- note added: "GND"
- note added: "PROGRAMMING HEADER"
- note removed: "DIM CONTROL DAC"
- note removed: "FTDI 5V\n"
- note removed: "FTDI GND"
- note removed: "FTDI PROGRAMMING HEADER"
- note removed: "FTDI RST"
- note removed: "FTDI RXD"
- note removed: "FTDI TXD"
- note removed: "FTDI/PWR 3V3"
- note removed: "FTDI/PWR GND"
- note removed: "RGB LED STATUS"
- moved on the sheet: R2, SW2

Commit message: PCB layout for v1.1.0 through hole prototype
Parts:
- removed C3: 22nF, Capacitor_THT:C_Radial_D4.0mm_H5.0mm_P1.50mm, symbol Device:C_Small
- removed C5, C6: 0.1µF, Capacitor_THT:C_Radial_D4.0mm_H5.0mm_P1.50mm, symbol Device:C_Small
- removed J3: Conn_01x08, symbol Connector_Generic:Conn_01x08
- added C1: 100nF, Capacitor_THT:CP_Radial_D5.0mm_P2.50mm, symbol Device:C_Small
- added C3: 4µ7, Capacitor_THT:CP_Radial_D5.0mm_P2.50mm, symbol Device:CP
- added C5: 0.1µ, Capacitor_THT:CP_Radial_D5.0mm_P2.50mm, symbol Device:CP
- added J3: Conn_02x04_Counter_Clockwise, Connector_PinSocket_2.54mm:PinSocket_2x04_P2.54mm_Vertical, symbol Connector_Generic:Conn_02x04_Counter_Clockwise
- BR1: symbol ceiling-light-dimmable-rescue:DB107-BP-Diode_Bridge_slimc-ceiling-light-dimmable-rescue -> ceiling-light-dimmable-rescue:DB107-BP-Diode_Bridge_slimc-ceiling-light-dimmable-rescue-ceiling-light-dimmable-rescue
- C2: footprint Capacitor_THT:C_Radial_D10.0mm_H12.5mm_P5.00mm -> Capacitor_THT:CP_Radial_D5.0mm_P2.50mm
- C4: footprint Capacitor_THT:C_Radial_D4.0mm_H5.0mm_P1.50mm -> Capacitor_THT:CP_Radial_D5.0mm_P2.50mm
- Q2, Q3: footprint Package_TO_SOT_THT:TO-220-3_Vertical -> Package_TO_SOT_SMD:TO-263-3_TabPin2
- Q4: footprint Package_TO_SOT_THT:TO-39-3 -> Package_TO_SOT_THT:TO-92_Inline
- R1, R11, R2, R5, R6, R9: footprint Resistor_SMD:R_1206_3216Metric_Pad1.42x1.75mm_HandSolder -> Resistor_THT:R_Axial_DIN0207_L6.3mm_D2.5mm_P10.16mm_Horizontal
- R10, R12, R13: value 2M -> 2M2; footprint Resistor_SMD:R_1206_3216Metric_Pad1.42x1.75mm_HandSolder -> Resistor_THT:R_Axial_DIN0411_L9.9mm_D3.6mm_P12.70mm_Horizontal
- SW1: footprint Button_Switch_THT:SW_PUSH_6mm -> Button_Switch_THT:SW_Tactile_Straight_KSA0Axx1LFTR
- SW2: footprint Button_Switch_SMD:SW_SPST_B3S-1000 -> Button_Switch_THT:SW_Tactile_Straight_KSA0Axx1LFTR
- U4: symbol ceiling-light-dimmable-rescue:FL51xxMX-AC_Drivers_slimc-ceiling-light-dimmable-rescue -> ceiling-light-dimmable-rescue:FL51xxMX-AC_Drivers_slimc-ceiling-light-dimmable-rescue-ceiling-light-dimmable-rescue
Connections:
- net DIM_MODE is gone; now on net ESP_GPIO_22: U4.4 (DM)
- net +3V3: now also C5.1, J3.6 (Pin_6)
- net +5V: now also J3.8 (Pin_8)
- net ESP_EN: now also J3.1 (Pin_1)
- net ESP_RXD0: now also J3.5 (Pin_5)
- net ESP_TXD0: now also J3.3 (Pin_3)
- net GND: now also C1.1, C3.2, C5.2, J3.2 (Pin_2), J3.4 (Pin_4)
- net N_MAIN: now also R13.2; no longer R13.1
- net at Q4.1 (E), U4.6 (VS): now also C3.1
- net at U4.1 (ZCMon): now also R13.1; no longer R13.2
- net ESP_GPIO_26: now reaches U6.11 (IO26)
- net ESP_GPIO_27: now reaches U6.12 (IO27)
- net ESP_GPIO_14: now reaches U6.13 (IO14)
- net ESP_GPIO_12: now reaches U6.14 (IO12)
- net ESP_GPIO_13: now reaches U6.16 (IO13)
- net ESP_GPIO_15: now reaches U6.23 (IO15)
- net ESP_GPIO_02: now reaches U6.24 (IO2)
- net ESP_GPIO_04: now reaches U6.26 (IO4)
- net ESP_GPIO_04: now also D1.4 (DIN)
- net ESP_GPIO_16: now reaches U6.27 (IO16)
- net ESP_GPIO_17: now reaches U6.28 (IO17)
- net ESP_GPIO_05: now reaches U6.29 (IO5)
- net ESP_GPIO_18: now reaches U6.30 (IO18)
- net ESP_GPIO_19: now reaches U6.31 (IO19)
- net ESP_GPIO_21: now reaches U6.33 (IO21)
- net ESP_GPIO_22: now reaches U6.36 (IO22)
- net ESP_GPIO_23: now reaches U6.37 (IO23)
- net ESP_GPIO_23: now also R2.1, U1.4
- net ESP_GPIO_35: now reaches U6.7 (IO35)
- net ESP_GPIO_35: now also U5.1 (Vout)
- net DIMCN renamed ESP_GPIO_25
- net ESP_GPIO_25: now also C1.2
- net ESP_GPIO0 renamed ESP_GPIO_00
- net ESP_GPIO_00: now also J3.7 (Pin_7)
- net LIGHT_SENSE renamed ESP_GPIO_34
- net ESP_GPIO_34: now also U6.6 (IO34); no longer U6.5 (SENSOR_VN)
- net M1_IN renamed L_M1
- net M2_IN renamed L_M2
- net STATUS_LED renamed ESP_GPIO_33
- net ESP_GPIO_33: no longer D1.4 (DIN)
- removed net SW_SENSE: R2.1, U1.4, U6.6 (IO34)
- net TEMP_SENSE renamed ESP_SENSOR_VP
- net ESP_SENSOR_VP: no longer U5.1 (Vout)
- new net ESP_SENSOR_VN: U6.5 (SENSOR_VN)
- no-connect marks 24 -> 22
Other:
- note added: "5 : GND"
- note added: "6 : GND"
- note added: "7 : 5V PWR"
- note added: "8 : 3V3 PWR"
- note added: "FTDI DTR -> ESP GPIO0 : 4"
- note added: "FTDI RTS -> ESP EN : 3"
- note added: "FTDI RXD -> ESP TXD : 1"
- note added: "FTDI TXD -> ESP RXD : 2"
- note removed: "3V3 PWR"
- note removed: "5V PWR"
- note removed: "FTDI DTR -> ESP GPIO0"
- note removed: "FTDI RTS -> ESP EN"
- note removed: "FTDI RXD -> ESP TXD"
- note removed: "FTDI TXD -> ESP RXD"
- note removed: "GND"
- moved on the sheet: BR1, C2, C4, D2, Q2, Q3, Q4, R1, R10, R11, R12, R13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
